Commit message: 2

File: source/My_quadruped_robot_lab/My_quadruped_robot_lab/assets/data/openrobot_wheelfixed/urdf/openrobot_wheelfixed.urdf (robot description, URDF)
Before this commit: robot openrobot_urdf_new_wheelfixed, 21 links, 20 joints
Joints:
- joint FL_calf_joint: limit lower=-0.3 upper=1.6 effort=300 velocity=9.4 -> lower=-0.6 upper=1.6 effort=300 velocity=9.4
- joint FR_calf_joint: limit lower=-1.6 upper=0.3 effort=300 velocity=9.4 -> lower=-1.6 upper=0.6 effort=300 velocity=9.4
- joint RL_calf_joint: limit lower=-0.3 upper=1.6 effort=300 velocity=9.4 -> lower=-0.6 upper=1.6 effort=300 velocity=9.4
- joint RR_calf_joint: limit lower=-1.6 upper=0.3 effort=300 velocity=9.4 -> lower=-1.6 upper=0.6 effort=300 velocity=9.4
